File: hardware/pcb/source/RaptorVR_1_0.kicad_pcb (KiCad board)
At the start: 2 copper layers, 86.4 x 53.3 mm, 16 parts, among them J3 LiPo wire pads, SW1 SK12D07VG3 high-3mm, U1 ELEGOO ESP-WROOM-32 USB-C 30-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, U2 MuMo V1.1 ICM-45686 + QMC6309, U3 TP4056 USB-C protected module

Commit message: Rename project to RaptorVR 1.0
Parts:
- removed the ? at (0.00, 0.00) (x6)
- added ?: , RaptorVR_1_0:NPTH_SW1_M1, F.Cu at (0.00, 0.00)
- added ?: , RaptorVR_1_0:NPTH_SW1_M2, F.Cu at (0.00, 0.00)
- added ?: , RaptorVR_1_0:NPTH_H_1, F.Cu at (0.00, 0.00)
- added ?: , RaptorVR_1_0:NPTH_H_2, F.Cu at (0.00, 0.00)
- added ?: , RaptorVR_1_0:NPTH_H_3, F.Cu at (0.00, 0.00)
- added ?: , RaptorVR_1_0:NPTH_H_4, F.Cu at (0.00, 0.00)
- D1: footprint PurrTrack32:D1 -> RaptorVR_1_0:D1
- D2: footprint PurrTrack32:D2 -> RaptorVR_1_0:D2
- J3: footprint PurrTrack32:J3 -> RaptorVR_1_0:J3
- R1: footprint PurrTrack32:R1 -> RaptorVR_1_0:R1
- R2: footprint PurrTrack32:R2 -> RaptorVR_1_0:R2
- R3: footprint PurrTrack32:R3 -> RaptorVR_1_0:R3
- SW1: footprint PurrTrack32:SW1 -> RaptorVR_1_0:SW1
- U1: footprint PurrTrack32:U1 -> RaptorVR_1_0:U1
- U2: footprint PurrTrack32:U2 -> RaptorVR_1_0:U2
- U3: footprint PurrTrack32:U3 -> RaptorVR_1_0:U3
Changed lines of the file:
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@@
-(kicad_pcb (version 20240108) (generator "PurrTrack32 generator")
+(kicad_pcb (version 20240108) (generator "RaptorVR 1.0 generator")
   (general (thickness 1.0))
   (paper "A4")
@@
   (net 13 "SYS_5V")
   (net 14 "USB_IN")
-  (footprint "PurrTrack32:U1" (layer "F.Cu") (at 0 0)
+  (footprint "RaptorVR_1_0:U1" (layer "F.Cu") (at 0 0)
     (property "Reference" "U1" (at 5.080 51.030 0) (layer "F.SilkS"))
     (property "Value" "ELEGOO ESP-WROOM-32 USB-C 30-pin" (at 5.080 3.580 0) (layer "F.Fab"))
@@
     (pad "R15" thru_hole circle (at 33.020 44.450) (size 1.800 1.800) (drill 1.000) (layers "*.Cu" "*.Mask") (net 10 "MOSI"))
   )
-  (footprint "PurrTrack32:U2" (layer "F.Cu") (at 0 0)
+  (footprint "RaptorVR_1_0:U2" (layer "F.Cu") (at 0 0)
     (property "Reference" "U2" (at 46.228 30.202 0) (layer "F.SilkS"))
     (property "Value" "MuMo V1.1 ICM-45686 + QMC6309" (at 46.228 12.470 0) (layer "F.Fab"))
@@
     (pad "6" thru_hole circle (at 61.468 14.732) (size 1.800 1.800) (drill 1.000) (layers "*.Cu" "*.Mask"))
   )
-  (footprint "PurrTrack32:U3" (layer "F.Cu") (at 0 0)
+  (footprint "RaptorVR_1_0:U3" (layer "F.Cu") (at 0 0)
     (property "Reference" "U3" (at 57.150 54.078 0) (layer "F.SilkS"))
     (property "Value" "TP4056 USB-C protected module" (at 57.150 34.822 0) (layer "F.Fab"))
@@
     (pad "7" thru_hole circle (at 58.166 39.116) (size 2.000 2.000) (drill 1.200) (layers "*.Cu" "*.Mask") (net 7 "GND"))
   )
-  (footprint "PurrTrack32:D1" (layer "F.Cu") (at 0 0)
+  (footprint "RaptorVR_1_0:D1" (layer "F.Cu") (at 0 0)
     (property "Reference" "D1" (at 64.008 33.758 0) (layer "F.SilkS"))
     (property "Value" "1N5817" (at 64.008 28.726 0) (layer "F.Fab"))
@@
     (pad "2" thru_hole circle (at 75.438 31.242) (size 2.200 2.200) (drill 1.000) (layers "*.Cu" "*.Mask") (net 11 "PWR_OR"))
   )
-  (footprint "PurrTrack32:D2" (layer "F.Cu") (at 0 0)
+  (footprint "RaptorVR_1_0:D2" (layer "F.Cu") (at 0 0)
     (property "Reference" "D2" (at 64.008 29.186 0) (layer "F.SilkS"))
     (property "Value" "1N5817" (at 64.008 24.154 0) (layer "F.Fab"))
@@
     (pad "2" thru_hole circle (at 75.438 26.670) (size 2.200 2.200) (drill 1.000) (layers "*.Cu" "*.Mask") (net 11 "PWR_OR"))
   )
-  (footprint "PurrTrack32:R1" (layer "F.Cu") (at 0 0)
+  (footprint "RaptorVR_1_0:R1" (layer "F.Cu") (at 0 0)
     (property "Reference" "R1" (at 37.084 48.744 0) (layer "F.SilkS"))
     (property "Value" "180k 1/4W" (at 37.084 43.712 0) (layer "F.Fab"))
@@
     (pad "2" thru_hole circle (at 48.260 46.228) (size 1.800 1.800) (drill 1.000) (layers "*.Cu" "*.Mask") (net 6 "DIV_A"))
   )
-  (footprint "PurrTrack32:R2" (layer "F.Cu") (at 0 0)
+  (footprint "RaptorVR_1_0:R2" (layer "F.Cu") (at 0 0)
     (property "Reference" "R2" (at 49.530 46.712 0) (layer "F.SilkS"))
     (property "Value" "220k 1/4W" (at 49.530 31.520 0) (layer "F.Fab"))
@@
     (pad "2" thru_hole circle (at 50.546 34.036) (size 1.800 1.800) (drill 1.000) (layers "*.Cu" "*.Mask") (net 2 "ADC_BAT"))
   )
-  (footprint "PurrTrack32:R3" (layer "F.Cu") (at 0 0)
+  (footprint "RaptorVR_1_0:R3" (layer "F.Cu") (at 0 0)
     (property "Reference" "R3" (at 37.338 34.520 0) (layer "F.SilkS"))
     (property "Value" "100k 1/4W" (at 37.338 29.488 0) (layer "F.Fab"))
@@
     (pad "2" thru_hole circle (at 48.514 32.004) (size 1.800 1.800) (drill 1.000) (layers "*.Cu" "*.Mask") (net 2 "ADC_BAT"))
   )
-  (footprint "PurrTrack32:SW1" (layer "F.Cu") (at 0 0)
+  (footprint "RaptorVR_1_0:SW1" (layer "F.Cu") (at 0 0)
     (property "Reference" "SW1" (at 72.644 22.328 0) (layer "F.SilkS"))
     (property "Value" "SK12D07VG3 high-3mm" (at 72.644 14.248 0) (layer "F.Fab"))
@@
     (pad "3" thru_hole circle (at 80.010 18.288) (size 2.200 2.200) (drill 1.100) (layers "*.Cu" "*.Mask") (net 13 "SYS_5V"))
   )
-  (footprint "PurrTrack32:J3" (layer "F.Cu") (at 0 0)
+  (footprint "RaptorVR_1_0:J3" (layer "F.Cu") (at 0 0)
     (property "Reference" "J3" (at 66.802 11.660 0) (layer "F.SilkS"))
     (property "Value" "LiPo wire pads" (at 66.802 4.596 0) (layer "F.Fab"))
@@
     (pad "-" thru_hole circle (at 76.200 8.128) (size 4.000 4.000) (drill 2.000) (layers "*.Cu" "*.Mask") (net 7 "GND"))
   )
-  (footprint "PurrTrack32:NPTH_SW1_M1" (layer "F.Cu") (at 0 0) (pad "" np_thru_hole circle (at 73.152 15.240) (size 1.800 1.800) (drill 1.800) (layers "*.Cu" "*.Mask")))
-  (footprint "PurrTrack32:NPTH_SW1_M2" (layer "F.Cu") (at 0 0) (pad "" np_thru_hole circle (at 81.788 15.240) (size 1.800 1.800) (drill 1.800) (layers "*.Cu" "*.Mask")))
-  (footprint "PurrTrack32:NPTH_H_1" (layer "F.Cu") (at 0 0) (pad "" np_thru_hole circle (at 3.810 3.810) (size 2.600 2.600) (drill 2.600) (layers "*.Cu" "*.Mask")))
-  (footprint "PurrTrack32:NPTH_H_2" (layer "F.Cu") (at 0 0) (pad "" np_thru_hole circle (at 82.550 3.810) (size 2.600 2.600) (drill 2.600) (layers "*.Cu" "*.Mask")))
-  (footprint "PurrTrack32:NPTH_H_3" (layer "F.Cu") (at 0 0) (pad "" np_thru_hole circle (at 3.810 49.530) (size 2.600 2.600) (drill 2.600) (layers "*.Cu" "*.Mask")))
-  (footprint "PurrTrack32:NPTH_H_4" (layer "F.Cu") (at 0 0) (pad "" np_thru_hole circle (at 53.340 49.530) (size 2.600 2.600) (drill 2.600) (layers "*.Cu" "*.Mask")))
+  (footprint "RaptorVR_1_0:NPTH_SW1_M1" (layer "F.Cu") (at 0 0) (pad "" np_thru_hole circle (at 73.152 15.240) (size 1.800 1.800) (drill 1.800) (layers "*.Cu" "*.Mask")))
+  (footprint "RaptorVR_1_0:NPTH_SW1_M2" (layer "F.Cu") (at 0 0) (pad "" np_thru_hole circle (at 81.788 15.240) (size 1.800 1.800) (drill 1.800) (layers "*.Cu" "*.Mask")))
+  (footprint "RaptorVR_1_0:NPTH_H_1" (layer "F.Cu") (at 0 0) (pad "" np_thru_hole circle (at 3.810 3.810) (size 2.600 2.600) (drill 2.600) (layers "*.Cu" "*.Mask")))
+  (footprint "RaptorVR_1_0:NPTH_H_2" (layer "F.Cu") (at 0 0) (pad "" np_thru_hole circle (at 82.550 3.810) (size 2.600 2.600) (drill 2.600) (layers "*.Cu" "*.Mask")))
+  (footprint "RaptorVR_1_0:NPTH_H_3" (layer "F.Cu") (at 0 0) (pad "" np_thru_hole circle (at 3.810 49.530) (size 2.600 2.600) (drill 2.600) (layers "*.Cu" "*.Mask")))
+  (footprint "RaptorVR_1_0:NPTH_H_4" (layer "F.Cu") (at 0 0) (pad "" np_thru_hole circle (at 53.340 49.530) (size 2.600 2.600) (drill 2.600) (layers "*.Cu" "*.Mask")))
   (segment (start 82.042 47.752) (end 65.278 47.752) (width 0.800) (layer "F.Cu") (net 14))
   (segment (start 65.278 47.752) (end 65.278 31.242) (width 0.800) (layer "F.Cu") (net 14))
